File: TM8-hardware/tm8_XP2.sch (EAGLE design)
At the start: 91 parts, among them IC1 MCP73831/OT, Q2 DMP1045U, U1 ATSAMD21G-A, U2 BME680, U3 SST25VF020BUSON, U4 LIS3DH, U5 DMG6968U-7, Y1 32.768kHz

Commit message: added beeps
Parts:
- removed C14: 0.1uF, rcl:C-EUC0402
- removed TP15, TP16, TP17: TPTP14R, testpad:TPTP14R
- removed U3: SST25VF020BUSON, SparkFun-IC-Memory:SST25VF020BUSON
- added IC2: 24LCS52ST, microchip:24LCS52ST
Connections:
- new net VN_UC: IC2.VCC
- net ALT: no longer TP17.TP, U3.SI
- net BTN2: no longer TP15.TP, U3.SCK
- net BTN4: no longer TP16.TP, U3.SO
- net GND: now also IC2.GND; no longer C14.2, U3.CE, U3.GND
- net SCL: now also IC2.SCL
- net SDA: now also IC2.SDA
- net VIN_UC: no longer C14.1, U3.HOLD, U3.VCC, U3.WP
Other:
- note removed: "TP15"
- note removed: "TP16"
- note removed: "TP17"
Changed lines of the file:
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@@
 <setting verticaltext="up"/>
 </settings>
-<grid distance="0.1" unitdist="inch" unit="inch" style="lines" multiple="1" display="no" altdistance="0.01" altunitdist="inch" altunit="inch"/>
+<grid distance="0.1" unitdist="inch" unit="inch" style="lines" multiple="1" display="yes" altdistance="0.01" altunitdist="inch" altunit="inch"/>
 <layers>
 <layer number="1" name="Top" color="4" fill="1" visible="no" active="no"/>
@@
 <part name="LS1" library="SMT-0340-T-R" deviceset="SMT-0340-T-R" device=""/>
 <part name="C17" library="rcl" library_urn="urn:adsk.eagle:library:334" deviceset="C-EU" device="C0402" package3d_urn="urn:adsk.eagle:package:23626/2" value="0.1uF"/>
-<part name="U3" library="SparkFun-IC-Memory" deviceset="SST25VF020B" device="USON"/>
 <part name="R1" library="adafruit" library_urn="urn:adsk.eagle:library:25768682" deviceset="R-US_" device="R0402" package3d_urn="urn:adsk.eagle:package:25769787/1"/>
 <part name="R2" library="adafruit" library_urn="urn:adsk.eagle:library:25768682" deviceset="R-US_" device="R0402" package3d_urn="urn:adsk.eagle:package:25769787/1"/>
@@
 <part name="TP6" library="testpad" library_urn="urn:adsk.eagle:library:385" deviceset="TP" device="TP14R" package3d_urn="urn:adsk.eagle:package:27966/1" value="TPTP14R"/>
 <part name="TP7" library="testpad" library_urn="urn:adsk.eagle:library:385" deviceset="TP" device="TP14R" package3d_urn="urn:adsk.eagle:package:27966/1" value="TPTP14R"/>
-<part name="C14" library="rcl" library_urn="urn:adsk.eagle:library:334" deviceset="C-EU" device="C0402" package3d_urn="urn:adsk.eagle:package:23626/2" value="0.1uF"/>
 <part name="TP8" library="testpad" library_urn="urn:adsk.eagle:library:385" deviceset="TP" device="TP14R" package3d_urn="urn:adsk.eagle:package:27966/1" value="TPTP14R"/>
 <part name="TP9" library="testpad" library_urn="urn:adsk.eagle:library:385" deviceset="TP" device="TP14R" package3d_urn="urn:adsk.eagle:package:27966/1" value="TPTP14R"/>
@@
 <part name="TP13" library="testpad" library_urn="urn:adsk.eagle:library:385" deviceset="TP" device="TP14R" package3d_urn="urn:adsk.eagle:package:27966/1" value="TPTP14R"/>
 <part name="TP14" library="testpad" library_urn="urn:adsk.eagle:library:385" deviceset="TP" device="TP14R" package3d_urn="urn:adsk.eagle:package:27966/1" value="TPTP14R"/>
-<part name="TP15" library="testpad" library_urn="urn:adsk.eagle:library:385" deviceset="TP" device="TP14R" package3d_urn="urn:adsk.eagle:package:27966/1" value="TPTP14R"/>
-<part name="TP16" library="testpad" library_urn="urn:adsk.eagle:library:385" deviceset="TP" device="TP14R" package3d_urn="urn:adsk.eagle:package:27966/1" value="TPTP14R"/>
-<part name="TP17" library="testpad" library_urn="urn:adsk.eagle:library:385" deviceset="TP" device="TP14R" package3d_urn="urn:adsk.eagle:package:27966/1" value="TPTP14R"/>
 <part name="TP18" library="testpad" library_urn="urn:adsk.eagle:library:385" deviceset="TP" device="TP14R" package3d_urn="urn:adsk.eagle:package:27966/1" value="TPTP14R"/>
+<part name="IC2" library="microchip" library_urn="urn:adsk.eagle:library:294" deviceset="24*" device="ST" package3d_urn="urn:adsk.eagle:package:20813/2" technology="LCS52"/>
 </parts>
 <sheets>
@@
 <text x="90.17" y="31.75" size="1.778" layer="95">TP13</text>
 <text x="90.17" y="29.21" size="1.778" layer="95">TP14</text>
-<text x="63.5" y="62.23" size="1.778" layer="95">TP15</text>
-<text x="63.5" y="59.69" size="1.778" layer="95">TP16</text>
-<text x="63.5" y="57.15" size="1.778" layer="95">TP17</text>
 <text x="63.5" y="68.58" size="1.778" layer="95">TP18</text>
 </plain>
@@
 <attribute name="VALUE" x="231.394" y="170.561" size="1.778" layer="96"/>
 </instance>
-<instance part="U3" gate="G$1" x="184.15" y="116.84" smashed="yes">
-<attribute name="NAME" x="173.99" y="122.174" size="1.778" layer="95" font="vector"/>
-<attribute name="VALUE" x="173.99" y="108.966" size="1.778" layer="96" font="vector" align="top-left"/>
-</instance>
 <instance part="R1" gate="G$1" x="179.07" y="144.78" smashed="yes">
 <attribute name="NAME" x="175.26" y="146.2786" size="1.778" layer="95"/>
@@
 <attribute name="TP_SIGNAL_NAME" x="62.23" y="72.39" size="1.778" layer="97" rot="R90"/>
 </instance>
-<instance part="C14" gate="G$1" x="212.09" y="119.38" smashed="yes" rot="R90">
-<attribute name="NAME" x="211.074" y="122.301" size="1.778" layer="95"/>
-<attribute name="VALUE" x="211.074" y="114.681" size="1.778" layer="96"/>
-</instance>
 <instance part="TP8" gate="G$1" x="87.63" y="46.99" smashed="yes" rot="R90">
 <attribute name="TP_SIGNAL_NAME" x="88.9" y="48.26" size="1.778" layer="97" rot="R90"/>
@@
 <attribute name="TP_SIGNAL_NAME" x="88.9" y="30.48" size="1.778" layer="97" rot="R90"/>
 </instance>
-<instance part="TP15" gate="G$1" x="60.96" y="62.23" smashed="yes" rot="R90">
-<attribute name="TP_SIGNAL_NAME" x="62.23" y="63.5" size="1.778" layer="97" rot="R90"/>
-</instance>
-<instance part="TP16" gate="G$1" x="60.96" y="59.69" smashed="yes" rot="R90">
-<attribute name="TP_SIGNAL_NAME" x="62.23" y="60.96" size="1.778" layer="97" rot="R90"/>
-</instance>
-<instance part="TP17" gate="G$1" x="60.96" y="57.15" smashed="yes" rot="R90">
-<attribute name="TP_SIGNAL_NAME" x="62.23" y="58.42" size="1.778" layer="97" rot="R90"/>
-</instance>
 <instance part="TP18" gate="G$1" x="60.96" y="68.58" smashed="yes" rot="R90">
 <attribute name="TP_SIGNAL_NAME" x="62.23" y="69.85" size="1.778" layer="97" rot="R90"/>
+</instance>
+<instance part="IC2" gate="G$1" x="185.42" y="119.38" smashed="yes" rot="R180">
+<attribute name="NAME" x="195.58" y="107.95" size="1.778" layer="95" rot="R180"/>
+<attribute name="VALUE" x="195.58" y="129.54" size="1.778" layer="96" rot="R180"/>
 </instance>
 </instances>
@@
 </segment>
 <segment>
-<pinref part="U3" gate="G$1" pin="GND"/>
-<wire x1="171.45" y1="111.76" x2="158.75" y2="111.76" width="0.1524" layer="91"/>
-<label x="158.75" y="111.76" size="1.778" layer="95"/>
-</segment>
-<segment>
 <pinref part="U5" gate="A" pin="S"/>
 <pinref part="R19" gate="G$1" pin="2"/>
@@
 </segment>
 <segment>
-<pinref part="C14" gate="G$1" pin="2"/>
-<wire x1="217.17" y1="119.38" x2="227.33" y2="119.38" width="0.1524" layer="91"/>
-<label x="222.25" y="119.38" size="1.778" layer="95"/>
-</segment>
-<segment>
-<pinref part="U3" gate="G$1" pin="CE"/>
-<wire x1="171.45" y1="119.38" x2="158.75" y2="119.38" width="0.1524" layer="91"/>
-<label x="158.75" y="119.38" size="1.778" layer="95"/>
+<pinref part="IC2" gate="G$1" pin="GND"/>
+<wire x1="177.8" y1="129.54" x2="157.48" y2="129.54" width="0.1524" layer="91"/>
+<label x="157.48" y="129.54" size="1.778" layer="95"/>
 </segment>
 </net>
@@
 <label x="229.87" y="33.02" size="1.778" layer="95"/>
 <pinref part="U1" gate="G$1" pin="PB11(SER4:3+)_SCK"/>
-</segment>
-<segment>
-<wire x1="209.55" y1="114.3" x2="196.85" y2="114.3" width="0.1524" layer="91"/>
-<pinref part="U3" gate="G$1" pin="SCK"/>
-<label x="196.85" y="114.3" size="1.778" layer="95"/>
-</segment>
-<segment>
-<pinref part="TP15" gate="G$1" pin="TP"/>
-<wire x1="63.5" y1="62.23" x2="80.01" y2="62.23" width="0.1524" layer="91"/>
-<label x="73.66" y="62.23" size="1.778" layer="95"/>
 </segment>
 </net>
@@
 <label x="99.06" y="46.99" size="1.778" layer="95"/>
 </segment>
+<segment>
+<pinref part="IC2" gate="G$1" pin="SCL"/>
+<wire x1="198.12" y1="111.76" x2="213.36" y2="111.76" width="0.1524" layer="91"/>
+<label x="208.28" y="111.76" size="1.778" layer="95"/>
+</segment>
 </net>
 <net name="SDA" class="0">
@@
 <label x="99.06" y="44.45" size="1.778" layer="95"/>
 </segment>
+<segment>
+<pinref part="IC2" gate="G$1" pin="SDA"/>
+<wire x1="170.18" y1="119.38" x2="157.48" y2="119.38" width="0.1524" layer="91"/>
+<label x="157.48" y="119.38" size="1.778" layer="95"/>
+</segment>
 </net>
 <net name="BTN3" class="0">
@@
 <label x="229.87" y="83.82" size="1.778" layer="95"/>
 <pinref part="U1" gate="G$1" pin="PA12(I2C/SER2:0+)_MISO"/>
-</segment>
-<segment>
-<pinref part="U3" gate="G$1" pin="SO"/>
-<wire x1="171.45" y1="116.84" x2="158.75" y2="116.84" width="0.1524" layer="91"/>
-<label x="158.75" y="116.84" size="1.778" layer="95"/>
-</segment>
-<segment>
-<pinref part="TP16" gate="G$1" pin="TP"/>
-<wire x1="63.5" y1="59.69" x2="80.01" y2="59.69" width="0.1524" layer="91"/>
-<label x="73.66" y="59.69" size="1.778" layer="95"/>
 </segment>
 </net>
@@
 <pinref part="U2" gate="G$1" pin="VDDIO"/>
 <wire x1="30.48" y1="97.79" x2="30.48" y2="102.87" width="0.1524" layer="91"/>
-</segment>
-<segment>
-<pinref part="U3" gate="G$1" pin="WP"/>
-<wire x1="171.45" y1="114.3" x2="158.75" y2="114.3" width="0.1524" layer="91"/>
-<label x="158.75" y="114.3" size="1.778" layer="95"/>
-</segment>
-<segment>
-<wire x1="209.55" y1="119.38" x2="196.85" y2="119.38" width="0.1524" layer="91"/>
-<pinref part="U3" gate="G$1" pin="VCC"/>
-<label x="196.85" y="119.38" size="1.778" layer="95"/>
-<pinref part="U3" gate="G$1" pin="HOLD"/>
-<wire x1="196.85" y1="116.84" x2="196.85" y2="119.38" width="0.1524" layer="91"/>
-<junction x="196.85" y="119.38"/>
-<pinref part="C14" gate="G$1" pin="1"/>
 </segment>
 <segment>
@@
 <label x="229.87" y="35.56" size="1.778" layer="95"/>
 </segment>
-<segment>
-<wire x1="209.55" y1="111.76" x2="196.85" y2="111.76" width="0.1524" layer="91"/>
-<pinref part="U3" gate="G$1" pin="SI"/>
-<label x="196.85" y="111.76" size="1.778" layer="95"/>
-</segment>
-<segment>
-<pinref part="TP17" gate="G$1" pin="TP"/>
-<wire x1="63.5" y1="57.15" x2="80.01" y2="57.15" width="0.1524" layer="91"/>
-<label x="73.66" y="57.15" size="1.778" layer="95"/>
-</segment>
 </net>
 <net name="N$17" class="0">
@@
 </segment>
 </net>
+<net name="VN_UC" class="0">
+<segment>
+<pinref part="IC2" gate="G$1" pin="VCC"/>
+<wire x1="177.8" y1="106.68" x2="157.48" y2="106.68" width="0.1524" layer="91"/>
+<label x="157.48" y="106.68" size="1.778" layer="95"/>
+</segment>
+</net>

Commit message: added sobriety game
Parts:
- added C14: 0.1uF, rcl:C-EUC0402
- added TP15, TP16: TPTP14R, testpad:TPTP14R
Connections:
- removed net VN_UC: IC2.VCC
- net GND: now also C14.2
- net SCL: no longer IC2.SCL
- net SCL1: now also IC2.SCL, TP15.TP
- net SDA: no longer IC2.SDA
- net SDA1: now also IC2.SDA, TP16.TP
- net VIN_UC: now also C14.1, IC2.VCC
Changed lines of the file:
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@@
 <setting verticaltext="up"/>
 </settings>
-<grid distance="0.1" unitdist="inch" unit="inch" style="lines" multiple="1" display="yes" altdistance="0.01" altunitdist="inch" altunit="inch"/>
+<grid distance="0.025" unitdist="inch" unit="inch" style="lines" multiple="1" display="yes" altdistance="0.01" altunitdist="inch" altunit="inch"/>
 <layers>
 <layer number="1" name="Top" color="4" fill="1" visible="no" active="no"/>
@@
 <part name="TP18" library="testpad" library_urn="urn:adsk.eagle:library:385" deviceset="TP" device="TP14R" package3d_urn="urn:adsk.eagle:package:27966/1" value="TPTP14R"/>
 <part name="IC2" library="microchip" library_urn="urn:adsk.eagle:library:294" deviceset="24*" device="ST" package3d_urn="urn:adsk.eagle:package:20813/2" technology="LCS52"/>
+<part name="TP15" library="testpad" library_urn="urn:adsk.eagle:library:385" deviceset="TP" device="TP14R" package3d_urn="urn:adsk.eagle:package:27966/1" value="TPTP14R"/>
+<part name="TP16" library="testpad" library_urn="urn:adsk.eagle:library:385" deviceset="TP" device="TP14R" package3d_urn="urn:adsk.eagle:package:27966/1" value="TPTP14R"/>
+<part name="C14" library="rcl" library_urn="urn:adsk.eagle:library:334" deviceset="C-EU" device="C0402" package3d_urn="urn:adsk.eagle:package:23626/2" value="0.1uF"/>
 </parts>
 <sheets>
@@
 <text x="90.17" y="29.21" size="1.778" layer="95">TP14</text>
 <text x="63.5" y="68.58" size="1.778" layer="95">TP18</text>
+<text x="209.55" y="127" size="1.778" layer="95">TP10</text>
+<text x="209.55" y="124.46" size="1.778" layer="95">TP11</text>
 </plain>
 <instances>
@@
 <attribute name="NAME" x="195.58" y="107.95" size="1.778" layer="95" rot="R180"/>
 <attribute name="VALUE" x="195.58" y="129.54" size="1.778" layer="96" rot="R180"/>
+</instance>
+<instance part="TP15" gate="G$1" x="207.01" y="127" smashed="yes" rot="R90">
+<attribute name="TP_SIGNAL_NAME" x="208.28" y="128.27" size="1.778" layer="97" rot="R90"/>
+</instance>
+<instance part="TP16" gate="G$1" x="207.01" y="124.46" smashed="yes" rot="R90">
+<attribute name="TP_SIGNAL_NAME" x="208.28" y="125.73" size="1.778" layer="97" rot="R90"/>
+</instance>
+<instance part="C14" gate="G$1" x="168.91" y="111.76" smashed="yes" rot="R180">
+<attribute name="NAME" x="167.386" y="111.379" size="1.778" layer="95" rot="R180"/>
+<attribute name="VALUE" x="167.386" y="116.459" size="1.778" layer="96" rot="R180"/>
 </instance>
 </instances>
@@
 <label x="157.48" y="129.54" size="1.778" layer="95"/>
 </segment>
+<segment>
+<pinref part="C14" gate="G$1" pin="2"/>
+<wire x1="168.91" y1="116.84" x2="157.48" y2="116.84" width="0.1524" layer="91"/>
+<label x="157.48" y="116.84" size="1.778" layer="95"/>
+</segment>
 </net>
 <net name="LED2" class="0">
@@
 <label x="99.06" y="46.99" size="1.778" layer="95"/>
 </segment>
-<segment>
-<pinref part="IC2" gate="G$1" pin="SCL"/>
-<wire x1="198.12" y1="111.76" x2="213.36" y2="111.76" width="0.1524" layer="91"/>
-<label x="208.28" y="111.76" size="1.778" layer="95"/>
-</segment>
 </net>
 <net name="SDA" class="0">
@@
 <wire x1="106.68" y1="44.45" x2="90.17" y2="44.45" width="0.1524" layer="91"/>
 <label x="99.06" y="44.45" size="1.778" layer="95"/>
-</segment>
-<segment>
-<pinref part="IC2" gate="G$1" pin="SDA"/>
-<wire x1="170.18" y1="119.38" x2="157.48" y2="119.38" width="0.1524" layer="91"/>
-<label x="157.48" y="119.38" size="1.778" layer="95"/>
 </segment>
 </net>
@@
 <wire x1="63.5" y1="68.58" x2="77.47" y2="68.58" width="0.1524" layer="91"/>
 <label x="73.66" y="68.58" size="1.778" layer="95"/>
+</segment>
+<segment>
+<pinref part="IC2" gate="G$1" pin="VCC"/>
+<wire x1="177.8" y1="106.68" x2="168.91" y2="106.68" width="0.1524" layer="91"/>
+<label x="157.48" y="106.68" size="1.778" layer="95"/>
+<pinref part="C14" gate="G$1" pin="1"/>
+<wire x1="168.91" y1="106.68" x2="157.48" y2="106.68" width="0.1524" layer="91"/>
+<wire x1="168.91" y1="109.22" x2="168.91" y2="106.68" width="0.1524" layer="91"/>
+<junction x="168.91" y="106.68"/>
 </segment>
 </net>
@@
 <label x="99.06" y="38.1" size="1.778" layer="95"/>
 </segment>
+<segment>
+<pinref part="IC2" gate="G$1" pin="SDA"/>
+<wire x1="170.18" y1="119.38" x2="157.48" y2="119.38" width="0.1524" layer="91"/>
+<label x="157.48" y="119.38" size="1.778" layer="95"/>
+</segment>
+<segment>
+<pinref part="TP16" gate="G$1" pin="TP"/>
+<wire x1="226.06" y1="124.46" x2="209.55" y2="124.46" width="0.1524" layer="91"/>
+<label x="218.44" y="124.46" size="1.778" layer="95"/>
+</segment>
 </net>
 <net name="SCL1" class="0">
@@
 <wire x1="90.17" y1="40.64" x2="106.68" y2="40.64" width="0.1524" layer="91"/>
 <label x="99.06" y="40.64" size="1.778" layer="95"/>
+</segment>
+<segment>
+<pinref part="IC2" gate="G$1" pin="SCL"/>
+<wire x1="198.12" y1="111.76" x2="213.36" y2="111.76" width="0.1524" layer="91"/>
+<label x="208.28" y="111.76" size="1.778" layer="95"/>
+</segment>
+<segment>
+<pinref part="TP15" gate="G$1" pin="TP"/>
+<wire x1="209.55" y1="127" x2="226.06" y2="127" width="0.1524" layer="91"/>
+<label x="218.44" y="127" size="1.778" layer="95"/>
 </segment>
 </net>
@@
 </segment>
 </net>
-<net name="VN_UC" class="0">
-<segment>
-<pinref part="IC2" gate="G$1" pin="VCC"/>
-<wire x1="177.8" y1="106.68" x2="157.48" y2="106.68" width="0.1524" layer="91"/>
-<label x="157.48" y="106.68" size="1.778" layer="95"/>
-</segment>
-</net>
